File: dual source.kicad_pcb (KiCad board)
At the start: 2 copper layers, 25.4 x 33 mm, 29 parts, among them P1 BATTERY, P2 CHRG, P3 CONN_01X08, P4 CONN_01X08, Q201 FDN340P, Q202 FDN340P, Q203 FDN340P, U1 SPX3819M5-3.3, U201 CN3063, U202 MCP6002

Commit message: So, having complete gnd plane helps...
Parts:
- C201, C204: value 10uF 16V -> 10uF
- C202: value 100nF 16V -> 100nF
- C203: value 100uF 16V X5R -> 100uF
- LED201: value LED_GREEN -> DONE
- LED202: value LED_RED -> CHRG
- R204, R205: value 7.15K 1% -> 7.15K
- U1: value SPX3819M5-3.3 -> SPX3819
- turned R204 to 270 degrees
Routing:
- net GND: track 0.00 -> 30.7 mm, vias 0 -> 5
- net Net-(R204-Pad1): track 7.42 -> 5.74 mm
Other:
- board text added: "+3V3"
- board text added: "+5V"
- board text added: "GND"
